Commit message: minor changes

File: rover.urdf (robot description, URDF)
Before this commit: robot rover, 22 links, 21 joints
Joints:
- joint joint_differential: limit lower=-0.524 upper=0.524 effort=10 velocity=1 -> lower=-0.3 upper=0.3 effort=10 velocity=1

Commit message: Add files via upload
added camera

File: rover.urdf (robot description, URDF)
Before this commit: robot rover, 22 links, 21 joints
Links:
- added link camera_link, mass 0.05; collision box size=0.04 0.10 0.03; visual box size=0.04 0.10 0.03
- added link camera_optical_link
Joints:
- added joint camera_joint: type fixed, parent base_link, child camera_link, origin xyz=0.425 0 0.1 rpy=0 0 0
- added joint camera_optical_joint: type fixed, parent camera_link, child camera_optical_link, origin xyz=0 0 0 rpy=-1.5708 0 -1.5708
