Commit message: Implement athena_sim simulation harness for IRC 2027
- Patch athena.urdf.xacro with sim:=true continuous wheel joints and collision/inertials
- Add athena_sim package with Gazebo Fortress DiffDrive and sensor plugins
- Add ros_gz_bridge config for clock, cmd_vel, RGB-D camera, IMU, and RTK GNSS
- Add sim_gps_rtk node with multi-mode RTK error model (Fixed/Float/Standalone/NoFix)
- Add vio_sim Option-B visual-inertial odometry drift and scale bias emulator
- Add procedural 120x120m Sproscape-Sim heightmap (PNG) and SDF world generator
- Add IRC 2027 mission clock, rules engine, proximity scorer, and briefing tool
- Add 3D SDF models for RADO tools, toolbox, delivery markers, red zones, and IDMO panel
- Add 28 unit tests passing with pure python unittest (no external ROS binary needed)

File: src/athena_gps_nav/urdf/athena.urdf.xacro (robot description, xacro)
@@ -1,4 +1,6 @@
 <?xml version="1.0"?>
 <robot xmlns:xacro="http://ros.org/wiki/xacro" name="athena">
+  <xacro:arg name="sim" default="false"/>
+  <xacro:property name="is_sim" value="$(arg sim)"/>
   <!--
     Athena rover description.
@@ -113,5 +115,26 @@
       <material name="athena_body"/>
     </visual>
-  </link>
+    <xacro:if value="${is_sim}">
+      <collision>
+        <geometry><box size="${base_length} ${base_width} ${base_thick}"/></geometry>
+      </collision>
+      <inertial>
+        <mass value="45.0"/>
+        <origin xyz="0 0 0" rpy="0 0 0"/>
+        <inertia ixx="${45.0 * (base_width*base_width + base_thick*base_thick) / 12.0}"
+                 ixy="0.0" ixz="0.0"
+                 iyy="${45.0 * (base_length*base_length + base_thick*base_thick) / 12.0}"
+                 iyz="0.0"
+                 izz="${45.0 * (base_length*base_length + base_width*base_width) / 12.0}"/>
+      </inertial>
+    </xacro:if>
+  </link>
+  <xacro:if value="${is_sim}">
+    <gazebo reference="base_link">
+      <material>Gazebo/DarkGrey</material>
+      <mu1>0.5</mu1>
+      <mu2>0.5</mu2>
+    </gazebo>
+  </xacro:if>
   <!-- base_link is the PARENT of base_footprint, not the child.  ekf_local
        publishes odom to base_link, so making base_footprint a parent would
@@ -134,4 +157,9 @@
       <material name="athena_accent"/>
     </visual>
+    <xacro:if value="${is_sim}">
+      <collision>
+        <geometry><box size="0.06 ${base_width * 0.6} 0.04"/></geometry>
+      </collision>
+    </xacro:if>
   </link>
   <joint name="nose_joint" type="fixed">
@@ -140,5 +168,5 @@
     <origin xyz="${base_length/2 - 0.02} 0 ${base_thick/2}" rpy="0 0 0"/>
   </joint>
-  <!-- ==== six wheels, visual only ======================================= -->
+  <!-- ==== six wheels ==================================================== -->
   <xacro:macro name="wheel" params="name x y">
     <link name="${name}">
@@ -147,11 +175,46 @@
         <material name="athena_wheel"/>
       </visual>
+      <xacro:if value="${is_sim}">
+        <collision>
+          <geometry><cylinder radius="${wheel_radius}" length="${wheel_width}"/></geometry>
+        </collision>
+        <inertial>
+          <mass value="2.5"/>
+          <origin xyz="0 0 0" rpy="0 0 0"/>
+          <inertia ixx="${2.5 * (3.0*wheel_radius*wheel_radius + wheel_width*wheel_width) / 12.0}"
+                   ixy="0.0" ixz="0.0"
+                   iyy="${2.5 * (3.0*wheel_radius*wheel_radius + wheel_width*wheel_width) / 12.0}"
+                   iyz="0.0"
+                   izz="${2.5 * wheel_radius * wheel_radius / 2.0}"/>
+        </inertial>
+      </xacro:if>
     </link>
-    <joint name="${name}_joint" type="fixed">
-      <parent link="base_link"/>
-      <child  link="${name}"/>
-      <!-- A cylinder's axis is +z and a wheel's axis is +y, hence the roll. -->
-      <origin xyz="${x} ${y} ${wheel_radius - base_height}" rpy="1.5708 0 0"/>
-    </joint>
+    <xacro:unless value="${is_sim}">
+      <joint name="${name}_joint" type="fixed">
+        <parent link="base_link"/>
+        <child  link="${name}"/>
+        <!-- A cylinder axis is +z and a wheel axis is +y, hence the roll. -->
+        <origin xyz="${x} ${y} ${wheel_radius - base_height}" rpy="1.5708 0 0"/>
+      </joint>
+    </xacro:unless>
+    <xacro:if value="${is_sim}">
+      <joint name="${name}_joint" type="continuous">
+        <parent link="base_link"/>
+        <child  link="${name}"/>
+        <!-- Local z after 90 deg roll points along base_link y (the spin axis) -->
+        <origin xyz="${x} ${y} ${wheel_radius - base_height}" rpy="1.5708 0 0"/>
+        <axis xyz="0 0 1"/>
+        <dynamics damping="0.05" friction="0.05"/>
+        <limit effort="40.0" velocity="20.0"/>
+      </joint>
+      <gazebo reference="${name}">
+        <material>Gazebo/Black</material>
+        <mu1>1.0</mu1>
+        <mu2>0.2</mu2>
+        <kp>1000000.0</kp>
+        <kd>100.0</kd>
+        <minDepth>0.005</minDepth>
+      </gazebo>
+    </xacro:if>
   </xacro:macro>
   <xacro:wheel name="wheel_front_left"  x="${wheel_x}"  y="${ track_width/2}"/>

Commit message: Update rover suspension to rocker-bogie and wheel diameter to 30cm
- Add rocker and bogie articulated suspension links with dynamic revolute joints
- Set wheel diameter to 30cm (radius 0.15m) and base_height ground clearance to 0.25m
- Set rocker-bogie main pivot axis 28cm below the depth camera (rocker_pivot_z = 0.27m)
- Update athena_sim DiffDrive plugin wheel_radius to 0.15m
- Add test_rocker_bogie_suspension_declared to unit test suite

File: src/athena_gps_nav/urdf/athena.urdf.xacro (robot description, xacro)
@@ -38,5 +38,5 @@
   <xacro:property name="base_length"  value="1.30"/>  <!-- x, front to back -->
   <xacro:property name="base_width"   value="1.00"/>  <!-- y, side to side  -->
-  <xacro:property name="base_height"  value="0.10"/>  <!-- ground to base_link -->
+  <xacro:property name="base_height"  value="0.25"/>  <!-- ground to base_link with 30cm wheels -->
   <xacro:property name="track_width"  value="0.85"/>  <!-- wheel centre to centre -->
   <!-- Camera: RealSense D435i, front centre.  Both numbers below are owner
@@ -100,9 +100,12 @@
   <xacro:property name="gps_y"        value="0.0"/>
   <xacro:property name="gps_z"        value="0.25"/>
-  <!-- Visual only, not measured. -->
-  <xacro:property name="base_thick"   value="0.12"/>
-  <xacro:property name="wheel_radius" value="0.06"/>
-  <xacro:property name="wheel_width"  value="0.04"/>
-  <xacro:property name="wheel_x"      value="0.45"/>   <!-- front/rear axle offset -->
+  <!-- Wheel dimensions: 30 cm diameter (radius 0.15 m), 8 cm width -->
+  <xacro:property name="base_thick"      value="0.12"/>
+  <xacro:property name="wheel_radius"    value="0.15"/>  <!-- 30 cm diameter -->
+  <xacro:property name="wheel_width"     value="0.08"/>  <!-- 8 cm width -->
+  <xacro:property name="wheel_x"         value="0.45"/>  <!-- front/rear axle offset -->
+  <!-- Rocker-Bogie main pivot: 28 cm below depth camera -->
+  <xacro:property name="rocker_pivot_x"  value="0.05"/>
+  <xacro:property name="rocker_pivot_z"  value="${camera_z - 0.28}"/>
   <material name="athena_body">  <color rgba="0.22 0.25 0.28 1.0"/></material>
   <material name="athena_accent"><color rgba="0.31 0.75 0.80 1.0"/></material>
@@ -168,6 +171,99 @@
     <origin xyz="${base_length/2 - 0.02} 0 ${base_thick/2}" rpy="0 0 0"/>
   </joint>
-  <!-- ==== six wheels ==================================================== -->
-  <xacro:macro name="wheel" params="name x y">
+  <!-- ==== rocker-bogie suspension and six wheels ====================== -->
+  <material name="athena_rocker"><color rgba="0.18 0.20 0.22 1.0"/></material>
+  <xacro:macro name="rocker_bogie_assembly" params="side y_sign">
+    <!-- Rocker link and main pivot joint -->
+    <link name="rocker_${side}">
+      <visual>
+        <!-- Beam from pivot forward to front wheel -->
+        <origin xyz="0.20 0 -0.185" rpy="0 0.74 0"/>
+        <geometry><box size="0.55 0.04 0.04"/></geometry>
+        <material name="athena_rocker"/>
+      </visual>
+      <visual>
+        <!-- Beam from pivot backward to bogie joint -->
+        <origin xyz="-0.10 0 -0.11" rpy="0 -0.83 0"/>
+        <geometry><box size="0.30 0.04 0.04"/></geometry>
+        <material name="athena_rocker"/>
+      </visual>
+      <xacro:if value="${is_sim}">
+        <collision>
+          <origin xyz="0.20 0 -0.185" rpy="0 0.74 0"/>
+          <geometry><box size="0.55 0.04 0.04"/></geometry>
+        </collision>
+        <inertial>
+          <mass value="3.0"/>
+          <origin xyz="0.10 0 -0.10" rpy="0 0 0"/>
+          <inertia ixx="0.02" ixy="0.0" ixz="0.0" iyy="0.08" iyz="0.0" izz="0.08"/>
+        </inertial>
+      </xacro:if>
+    </link>
+    <xacro:unless value="${is_sim}">
+      <joint name="rocker_${side}_joint" type="fixed">
+        <parent link="base_link"/>
+        <child  link="rocker_${side}"/>
+        <origin xyz="${rocker_pivot_x} ${y_sign * track_width/2} ${rocker_pivot_z}" rpy="0 0 0"/>
+      </joint>
+    </xacro:unless>
+    <xacro:if value="${is_sim}">
+      <joint name="rocker_${side}_joint" type="revolute">
+        <parent link="base_link"/>
+        <child  link="rocker_${side}"/>
+        <origin xyz="${rocker_pivot_x} ${y_sign * track_width/2} ${rocker_pivot_z}" rpy="0 0 0"/>
+        <axis xyz="0 1 0"/>
+        <limit lower="-0.45" upper="0.45" effort="120.0" velocity="5.0"/>
+        <dynamics damping="1.0" friction="0.5"/>
+      </joint>
+    </xacro:if>
+    <!-- Bogie link and pivot joint -->
+    <link name="bogie_${side}">
+      <visual>
+        <!-- Beam from bogie pivot forward to mid wheel and rear to back wheel -->
+        <origin xyz="-0.075 0 -0.075" rpy="0 0.0 0"/>
+        <geometry><box size="0.48 0.04 0.04"/></geometry>
+        <material name="athena_rocker"/>
+      </visual>
+      <xacro:if value="${is_sim}">
+        <collision>
+          <origin xyz="-0.075 0 -0.075" rpy="0 0.0 0"/>
+          <geometry><box size="0.48 0.04 0.04"/></geometry>
+        </collision>
+        <inertial>
+          <mass value="2.5"/>
+          <origin xyz="-0.075 0 -0.075" rpy="0 0 0"/>
+          <inertia ixx="0.015" ixy="0.0" ixz="0.0" iyy="0.05" iyz="0.0" izz="0.05"/>
+        </inertial>
+      </xacro:if>
+    </link>
+    <xacro:unless value="${is_sim}">
+      <joint name="bogie_${side}_joint" type="fixed">
+        <parent link="rocker_${side}"/>
+        <child  link="bogie_${side}"/>
+        <origin xyz="-0.20 0.0 -0.22" rpy="0 0 0"/>
+      </joint>
+    </xacro:unless>
+    <xacro:if value="${is_sim}">
+      <joint name="bogie_${side}_joint" type="revolute">
+        <parent link="rocker_${side}"/>
+        <child  link="bogie_${side}"/>
+        <origin xyz="-0.20 0.0 -0.22" rpy="0 0 0"/>
+        <axis xyz="0 1 0"/>
+        <limit lower="-0.45" upper="0.45" effort="100.0" velocity="5.0"/>
+        <dynamics damping="1.0" friction="0.5"/>
+      </joint>
+    </xacro:if>
+    <!-- Front Wheel attached to Rocker -->
+    <xacro:wheel_instance name="wheel_front_${side}" parent="rocker_${side}"
+                          x="0.40" y="0.0" z="-0.37"/>
+    <!-- Mid Wheel attached to Bogie -->
+    <xacro:wheel_instance name="wheel_mid_${side}" parent="bogie_${side}"
+                          x="0.15" y="0.0" z="-0.15"/>
+    <!-- Rear Wheel attached to Bogie -->
+    <xacro:wheel_instance name="wheel_rear_${side}" parent="bogie_${side}"
+                          x="-0.30" y="0.0" z="-0.15"/>
+  </xacro:macro>
+  <!-- Wheel instance macro (30 cm diameter, 3.5 kg mass) -->
+  <xacro:macro name="wheel_instance" params="name parent x y z">
     <link name="${name}">
       <visual>
@@ -180,11 +276,9 @@
         </collision>
         <inertial>
-          <mass value="2.5"/>
+          <mass value="3.5"/>
           <origin xyz="0 0 0" rpy="0 0 0"/>
-          <inertia ixx="${2.5 * (3.0*wheel_radius*wheel_radius + wheel_width*wheel_width) / 12.0}"
-                   ixy="0.0" ixz="0.0"
-                   iyy="${2.5 * (3.0*wheel_radius*wheel_radius + wheel_width*wheel_width) / 12.0}"
-                   iyz="0.0"
-                   izz="${2.5 * wheel_radius * wheel_radius / 2.0}"/>
+          <inertia ixx="0.0215" ixy="0.0" ixz="0.0"
+                   iyy="0.0215" iyz="0.0"
+                   izz="0.0394"/>
         </inertial>
       </xacro:if>
@@ -192,19 +286,17 @@
     <xacro:unless value="${is_sim}">
       <joint name="${name}_joint" type="fixed">
-        <parent link="base_link"/>
+        <parent link="${parent}"/>
         <child  link="${name}"/>
-        <!-- A cylinder axis is +z and a wheel axis is +y, hence the roll. -->
-        <origin xyz="${x} ${y} ${wheel_radius - base_height}" rpy="1.5708 0 0"/>
+        <origin xyz="${x} ${y} ${z}" rpy="1.5708 0 0"/>
       </joint>
     </xacro:unless>
     <xacro:if value="${is_sim}">
       <joint name="${name}_joint" type="continuous">
-        <parent link="base_link"/>
+        <parent link="${parent}"/>
         <child  link="${name}"/>
-        <!-- Local z after 90 deg roll points along base_link y (the spin axis) -->
-        <origin xyz="${x} ${y} ${wheel_radius - base_height}" rpy="1.5708 0 0"/>
+        <origin xyz="${x} ${y} ${z}" rpy="1.5708 0 0"/>
         <axis xyz="0 0 1"/>
-        <dynamics damping="0.05" friction="0.05"/>
-        <limit effort="40.0" velocity="20.0"/>
+        <dynamics damping="0.08" friction="0.05"/>
+        <limit effort="50.0" velocity="20.0"/>
       </joint>
       <gazebo reference="${name}">
@@ -218,10 +310,6 @@
     </xacro:if>
   </xacro:macro>
-  <xacro:wheel name="wheel_front_left"  x="${wheel_x}"  y="${ track_width/2}"/>
-  <xacro:wheel name="wheel_front_right" x="${wheel_x}"  y="${-track_width/2}"/>
-  <xacro:wheel name="wheel_mid_left"    x="0"           y="${ track_width/2}"/>
-  <xacro:wheel name="wheel_mid_right"   x="0"           y="${-track_width/2}"/>
-  <xacro:wheel name="wheel_rear_left"   x="${-wheel_x}" y="${ track_width/2}"/>
-  <xacro:wheel name="wheel_rear_right"  x="${-wheel_x}" y="${-track_width/2}"/>
+  <xacro:rocker_bogie_assembly side="left"  y_sign="1"/>
+  <xacro:rocker_bogie_assembly side="right" y_sign="-1"/>
   <!-- ==== sensors ======================================================= -->
   <!-- The RealSense driver hangs its own optical frames under camera_link

File: src/athena_sim/urdf/athena_sim.urdf.xacro (robot description, xacro)
@@ -25,5 +25,5 @@
       <right_joint>wheel_rear_right_joint</right_joint>
       <wheel_separation>0.85</wheel_separation>
-      <wheel_radius>0.06</wheel_radius>
+      <wheel_radius>0.15</wheel_radius>
       <odom_publish_frequency>20</odom_publish_frequency>
       <topic>/cmd_vel</topic>
