Commit message: feat(sim): improve rover rocker-bogie URDF, center terrain at origin z=0, and remove start gate

File: src/athena_gps_nav/urdf/athena.urdf.xacro (robot description, xacro)
@@ -34,58 +34,20 @@
        with a symlink install (see CONTRIBUTING.md) and relaunch.
        ===================================================================== -->
-  <!-- Chassis. Tape measured 2026-09-02, and it agrees with both
-       athena_drive's saved track_width and nav2_params' footprint. -->
-  <xacro:property name="base_length"  value="1.30"/>  <!-- x, front to back -->
-  <xacro:property name="base_width"   value="1.00"/>  <!-- y, side to side  -->
-  <xacro:property name="base_height"  value="0.25"/>  <!-- ground to base_link with 30cm wheels -->
-  <xacro:property name="track_width"  value="0.85"/>  <!-- wheel centre to centre -->
-  <!-- Camera: RealSense D435i, front centre.  Both numbers below are owner
-       tape measurements, 2026-09-03: the lens is 0.50 m forward of the
-       chassis centre (so 0.15 m back from the front face) and 0.65 m above
-       the ground, hence camera_z = 0.65 - base_height.
-       camera_x was 0.10 until 2026-09-03, i.e. 0.40 m behind where the lens
-       actually is.  Every depth point was marked that much closer to the
-       rover than it really was, so returns from just past the front bumper
-       landed INSIDE the Nav2 footprint and the controller read them as a
-       collision it could not drive out of. -->
+  <!-- Chassis. Measured for Athena competition rover:
+       Avionics/chassis box is 28cm high, 54cm wide, 85cm long.
+       Base_link is origin; ground is at -base_height = -0.25m. -->
+  <xacro:property name="base_length"     value="0.85"/>  <!-- x, front to back -->
+  <xacro:property name="base_width"      value="0.54"/>  <!-- y, side to side  -->
+  <xacro:property name="base_height"     value="0.25"/>  <!-- ground to base_link with 30cm wheels -->
+  <xacro:property name="chassis_height"  value="0.28"/>  <!-- 28 cm chassis box height -->
+  <xacro:property name="track_width"     value="0.85"/>  <!-- wheel centre to centre -->
+  <!-- Camera: RealSense D435i mounted at top of chassis at front centre.
+       Lens is at x = 0.50 (front face of chassis), z = 0.40 (top deck of chassis,
+       which sits 0.65 m above the ground: 0.40 - (-0.25) = 0.65 m). -->
   <xacro:property name="camera_x"     value="0.50"/>
-  <xacro:property name="camera_z"     value="0.55"/>
-  <!-- Camera tilt about its own left axis, radians.  ROS sign convention:
-       POSITIVE pitch is nose DOWN.  A lot of the confusion in this file's
-       history came from getting that backwards.
-       0.0 because the camera is currently mounted level, in normal
-       landscape (owner, 2026-09-03).
-       This was -0.10 until 2026-09-03, i.e. the model believed the camera
-       was tilted 5.7 degrees UP when it is in fact level.  That rotates
-       every depth point upward by the same angle, and the error grows with
-       range: the floor 2 m ahead of the lens lands at z = +0.10 m in
-       base_link instead of -0.10 m, which is exactly min_obstacle_height.
-       So flat ground from about 2 m out was being marked LETHAL, in a
-       band right across the camera's field of view.  Together with the
-       camera_x error that band sat about 2 m in front of the bumper, the
-       controller refused to drive into it, and Nav2 fell through to its
-       Spin recovery, which turns 1.57 rad to the left.
-       WHEN YOU TILT THE CAMERA DOWN (planned, to spot low objects like a
-       hammer near the wheels): put the REAL angle here as a POSITIVE
-       number, and measure it, do not eyeball it.  Guessing brings the
-       phantom wall straight back, and a downward tilt makes it worse
-       because more of the frame is floor.  Run
-       indoor_test/mount_check.py camera after remounting; it reads the
-       tilt off the floor plane and prints the value to paste here.
-       Note also that min_obstacle_height (0.10 m in nav2_params.yaml) sits
-       0.20 m above the ground, so a hammer will still be invisible until
-       that is lowered as well.  Lower it only once this angle is measured,
-       not before, or you will be marking the floor on purpose. -->
+  <xacro:property name="camera_z"     value="0.40"/>
+  <!-- Camera tilt about its own left axis, radians. 0.0 for level mounting. -->
   <xacro:property name="camera_pitch" value="0.0"/>
-  <!-- Pixhawk: same place as the camera, 15 cm lower (owner, 2026-09-03).
-       Only the ORIENTATION of this frame affects navigation: the EKF rotates
-       the gyro into base_link with it, and fuses yaw rate.  The translation
-       is cosmetic here because no accelerometer channel is fused, but it is
-       written honestly so nobody has to re-derive it later.
-       imu_rpy is zero, which asserts the board is bolted down flat with its
-       forward arrow pointing at the front of the rover.  If it is rotated or
-       inverted, put the real angles here, because a Pixhawk mounted upside
-       down reports yaw rate with the wrong sign and the rover will turn away
-       from its goal instead of toward it. -->
+  <!-- Pixhawk IMU: inside front avionics bay, 15 cm below depth camera. -->
   <xacro:property name="imu_x"        value="${camera_x}"/>
   <xacro:property name="imu_z"        value="${camera_z - 0.15}"/>
@@ -93,41 +55,53 @@
   <xacro:property name="imu_pitch"    value="0.0"/>
   <xacro:property name="imu_yaw"      value="0.0"/>
-  <!-- GPS antenna, relative to base_link.  navsat_transform uses this to
-       remove the antenna lever arm from the fix.  NOT YET MEASURED: it is a
-       guess that the antenna is over the chassis centre.  Harmless for local
-       obstacle avoidance, worth a tape measure before waypoint work. -->
+  <!-- GPS antenna: mounted on top deck of chassis at z = 0.41 m. -->
   <xacro:property name="gps_x"        value="0.0"/>
   <xacro:property name="gps_y"        value="0.0"/>
-  <xacro:property name="gps_z"        value="0.25"/>
+  <xacro:property name="gps_z"        value="${camera_z + 0.01}"/>
   <!-- Wheel dimensions: 30 cm diameter (radius 0.15 m), 8 cm width -->
-  <xacro:property name="base_thick"      value="0.12"/>
   <xacro:property name="wheel_radius"    value="0.15"/>  <!-- 30 cm diameter -->
   <xacro:property name="wheel_width"     value="0.08"/>  <!-- 8 cm width -->
   <xacro:property name="wheel_x"         value="0.45"/>  <!-- front/rear axle offset -->
-  <!-- Rocker-Bogie main pivot: 28 cm below depth camera -->
+  <!-- Rocker-Bogie main pivot: at the lower end of the chassis (28 cm below camera) -->
   <xacro:property name="rocker_pivot_x"  value="0.05"/>
-  <xacro:property name="rocker_pivot_z"  value="${camera_z - 0.28}"/>
+  <xacro:property name="rocker_pivot_z"  value="${camera_z - chassis_height}"/>
   <material name="athena_body">  <color rgba="0.22 0.25 0.28 1.0"/></material>
   <material name="athena_accent"><color rgba="0.31 0.75 0.80 1.0"/></material>
   <material name="athena_wheel"> <color rgba="0.10 0.10 0.11 1.0"/></material>
   <material name="athena_gps">   <color rgba="0.95 0.72 0.20 1.0"/></material>
+  <material name="athena_rocker"><color rgba="0.18 0.20 0.22 1.0"/></material>
   <!-- ==== chassis ======================================================= -->
   <link name="base_link">
-    <visual>
-      <geometry><box size="${base_length} ${base_width} ${base_thick}"/></geometry>
+    <!-- Main central avionics & battery chassis body (28cm high) -->
+    <visual>
+      <origin xyz="0.075 0 0.26" rpy="0 0 0"/>
+      <geometry><box size="${base_length} ${base_width} ${chassis_height}"/></geometry>
       <material name="athena_body"/>
     </visual>
+    <!-- Top equipment deck -->
+    <visual>
+      <origin xyz="0.05 0 0.401" rpy="0 0 0"/>
+      <geometry><box size="0.75 0.50 0.005"/></geometry>
+      <material name="athena_accent"/>
+    </visual>
+    <!-- Transverse rocker pivot axle tube extending across lower end of chassis -->
+    <visual>
+      <origin xyz="${rocker_pivot_x} 0 ${rocker_pivot_z}" rpy="1.5708 0 0"/>
+      <geometry><cylinder radius="0.025" length="${track_width}"/></geometry>
+      <material name="athena_rocker"/>
+    </visual>
     <xacro:if value="${is_sim}">
       <collision>
-        <geometry><box size="${base_length} ${base_width} ${base_thick}"/></geometry>
+        <origin xyz="0.075 0 0.26" rpy="0 0 0"/>
+        <geometry><box size="${base_length} ${base_width} ${chassis_height}"/></geometry>
       </collision>
       <inertial>
-        <mass value="45.0"/>
-        <origin xyz="0 0 0" rpy="0 0 0"/>
-        <inertia ixx="${45.0 * (base_width*base_width + base_thick*base_thick) / 12.0}"
+        <mass value="35.0"/>
+        <origin xyz="0.05 0 0.24" rpy="0 0 0"/>
+        <inertia ixx="${35.0 * (base_width*base_width + chassis_height*chassis_height) / 12.0}"
                  ixy="0.0" ixz="0.0"
-                 iyy="${45.0 * (base_length*base_length + base_thick*base_thick) / 12.0}"
+                 iyy="${35.0 * (base_length*base_length + chassis_height*chassis_height) / 12.0}"
                  iyz="0.0"
-                 izz="${45.0 * (base_length*base_length + base_width*base_width) / 12.0}"/>
+                 izz="${35.0 * (base_length*base_length + base_width*base_width) / 12.0}"/>
       </inertial>
     </xacro:if>
@@ -140,10 +114,4 @@
     </gazebo>
   </xacro:if>
-  <!-- base_link is the PARENT of base_footprint, not the child.  ekf_local
-       publishes odom to base_link, so making base_footprint a parent would
-       give base_link two parents.  TF2 requires exactly one, and the result
-       is that base_footprint gets orphaned and every lookup involving it
-       throws ConnectivityException.  That bites because Nav2 configs
-       commonly use base_footprint as robot_base_frame. -->
   <link name="base_footprint"/>
   <joint name="base_footprint_joint" type="fixed">
@@ -152,15 +120,13 @@
     <origin xyz="0 0 ${-base_height}" rpy="0 0 0"/>
   </joint>
-  <!-- A nose block, so "forward" is unmistakable in a 3D view.  A bare box
-       looks the same from both ends and you cannot tell a reversing rover
-       from an advancing one. -->
+  <!-- Front nose marker block for unmistakable orientation -->
   <link name="nose_marker">
     <visual>
-      <geometry><box size="0.06 ${base_width * 0.6} 0.04"/></geometry>
+      <geometry><box size="0.04 ${base_width * 0.7} 0.08"/></geometry>
       <material name="athena_accent"/>
     </visual>
     <xacro:if value="${is_sim}">
       <collision>
-        <geometry><box size="0.06 ${base_width * 0.6} 0.04"/></geometry>
+        <geometry><box size="0.04 ${base_width * 0.7} 0.08"/></geometry>
       </collision>
     </xacro:if>
@@ -169,31 +135,42 @@
     <parent link="base_link"/>
     <child  link="nose_marker"/>
-    <origin xyz="${base_length/2 - 0.02} 0 ${base_thick/2}" rpy="0 0 0"/>
+    <origin xyz="0.51 0 0.32" rpy="0 0 0"/>
   </joint>
   <!-- ==== rocker-bogie suspension and six wheels ====================== -->
-  <material name="athena_rocker"><color rgba="0.18 0.20 0.22 1.0"/></material>
   <xacro:macro name="rocker_bogie_assembly" params="side y_sign">
     <!-- Rocker link and main pivot joint -->
     <link name="rocker_${side}">
-      <visual>
-        <!-- Beam from pivot forward to front wheel -->
-        <origin xyz="0.20 0 -0.185" rpy="0 0.74 0"/>
-        <geometry><box size="0.55 0.04 0.04"/></geometry>
-        <material name="athena_rocker"/>
-      </visual>
-      <visual>
-        <!-- Beam from pivot backward to bogie joint -->
-        <origin xyz="-0.10 0 -0.11" rpy="0 -0.83 0"/>
-        <geometry><box size="0.30 0.04 0.04"/></geometry>
+      <!-- Pivot hub cylinder -->
+      <visual>
+        <origin xyz="0 0 0" rpy="1.5708 0 0"/>
+        <geometry><cylinder radius="0.035" length="0.06"/></geometry>
+        <material name="athena_rocker"/>
+      </visual>
+      <!-- Beam from pivot forward and down to front wheel -->
+      <visual>
+        <origin xyz="0.20 0 -0.11" rpy="0 0.502 0"/>
+        <geometry><box size="0.456 0.04 0.04"/></geometry>
+        <material name="athena_rocker"/>
+      </visual>
+      <!-- Beam from pivot backward and down to bogie joint -->
+      <visual>
+        <origin xyz="-0.10 0 -0.06" rpy="0 -0.540 0"/>
+        <geometry><box size="0.233 0.04 0.04"/></geometry>
+        <material name="athena_rocker"/>
+      </visual>
+      <!-- Bogie joint housing hub -->
+      <visual>
+        <origin xyz="-0.20 0 -0.12" rpy="1.5708 0 0"/>
+        <geometry><cylinder radius="0.03" length="0.05"/></geometry>
         <material name="athena_rocker"/>
       </visual>
       <xacro:if value="${is_sim}">
         <collision>
-          <origin xyz="0.20 0 -0.185" rpy="0 0.74 0"/>
-          <geometry><box size="0.55 0.04 0.04"/></geometry>
+          <origin xyz="0.20 0 -0.11" rpy="0 0.502 0"/>
+          <geometry><box size="0.456 0.04 0.04"/></geometry>
         </collision>
         <inertial>
           <mass value="3.0"/>
-          <origin xyz="0.10 0 -0.10" rpy="0 0 0"/>
+          <origin xyz="0.10 0 -0.08" rpy="0 0 0"/>
           <inertia ixx="0.02" ixy="0.0" ixz="0.0" iyy="0.08" iyz="0.0" izz="0.08"/>
         </inertial>
@@ -219,18 +196,30 @@
     <!-- Bogie link and pivot joint -->
     <link name="bogie_${side}">
-      <visual>
-        <!-- Beam from bogie pivot forward to mid wheel and rear to back wheel -->
-        <origin xyz="-0.075 0 -0.075" rpy="0 0.0 0"/>
-        <geometry><box size="0.48 0.04 0.04"/></geometry>
+      <!-- Bogie center pivot hub -->
+      <visual>
+        <origin xyz="0 0 0" rpy="1.5708 0 0"/>
+        <geometry><cylinder radius="0.03" length="0.055"/></geometry>
+        <material name="athena_rocker"/>
+      </visual>
+      <!-- Beam from bogie pivot forward and down to mid wheel -->
+      <visual>
+        <origin xyz="0.075 0 -0.05" rpy="0 0.588 0"/>
+        <geometry><box size="0.18 0.035 0.035"/></geometry>
+        <material name="athena_rocker"/>
+      </visual>
+      <!-- Beam from bogie pivot backward and down to rear wheel -->
+      <visual>
+        <origin xyz="-0.15 0 -0.05" rpy="0 -0.322 0"/>
+        <geometry><box size="0.316 0.035 0.035"/></geometry>
         <material name="athena_rocker"/>
       </visual>
       <xacro:if value="${is_sim}">
         <collision>
-          <origin xyz="-0.075 0 -0.075" rpy="0 0.0 0"/>
-          <geometry><box size="0.48 0.04 0.04"/></geometry>
+          <origin xyz="-0.075 0 -0.05" rpy="0 0 0"/>
+          <geometry><box size="0.48 0.035 0.035"/></geometry>
         </collision>
         <inertial>
           <mass value="2.5"/>
-          <origin xyz="-0.075 0 -0.075" rpy="0 0 0"/>
+          <origin xyz="-0.075 0 -0.05" rpy="0 0 0"/>
           <inertia ixx="0.015" ixy="0.0" ixz="0.0" iyy="0.05" iyz="0.0" izz="0.05"/>
         </inertial>
@@ -241,5 +230,5 @@
         <parent link="rocker_${side}"/>
         <child  link="bogie_${side}"/>
-        <origin xyz="-0.20 0.0 -0.22" rpy="0 0 0"/>
+        <origin xyz="-0.20 0.0 -0.12" rpy="0 0 0"/>
       </joint>
     </xacro:unless>
@@ -248,5 +237,5 @@
         <parent link="rocker_${side}"/>
         <child  link="bogie_${side}"/>
-        <origin xyz="-0.20 0.0 -0.22" rpy="0 0 0"/>
+        <origin xyz="-0.20 0.0 -0.12" rpy="0 0 0"/>
         <axis xyz="0 1 0"/>
         <limit lower="-0.45" upper="0.45" effort="100.0" velocity="5.0"/>
@@ -254,20 +243,26 @@
       </joint>
     </xacro:if>
-    <!-- Front Wheel attached to Rocker -->
+    <!-- Front Wheel attached to Rocker (x=0.45, z=-0.10 in base_link) -->
     <xacro:wheel_instance name="wheel_front_${side}" parent="rocker_${side}"
-                          x="0.40" y="0.0" z="-0.37"/>
-    <!-- Mid Wheel attached to Bogie -->
+                          x="0.40" y="0.0" z="-0.22"/>
+    <!-- Mid Wheel attached to Bogie (x=0.00, z=-0.10 in base_link) -->
     <xacro:wheel_instance name="wheel_mid_${side}" parent="bogie_${side}"
-                          x="0.15" y="0.0" z="-0.15"/>
-    <!-- Rear Wheel attached to Bogie -->
+                          x="0.15" y="0.0" z="-0.10"/>
+    <!-- Rear Wheel attached to Bogie (x=-0.45, z=-0.10 in base_link) -->
     <xacro:wheel_instance name="wheel_rear_${side}" parent="bogie_${side}"
-                          x="-0.30" y="0.0" z="-0.15"/>
+                          x="-0.30" y="0.0" z="-0.10"/>
   </xacro:macro>
   <!-- Wheel instance macro (30 cm diameter, 3.5 kg mass) -->
   <xacro:macro name="wheel_instance" params="name parent x y z">
     <link name="${name}">
+      <!-- Outer treaded tire -->
       <visual>
         <geometry><cylinder radius="${wheel_radius}" length="${wheel_width}"/></geometry>
         <material name="athena_wheel"/>
+      </visual>
+      <!-- Inner accent hubcap -->
+      <visual>
+        <geometry><cylinder radius="${wheel_radius * 0.60}" length="${wheel_width + 0.004}"/></geometry>
+        <material name="athena_accent"/>
       </visual>
       <xacro:if value="${is_sim}">
@@ -313,12 +308,17 @@
   <xacro:rocker_bogie_assembly side="right" y_sign="-1"/>
   <!-- ==== sensors ======================================================= -->
-  <!-- The RealSense driver hangs its own optical frames under camera_link
-       (via the camera_link to camera_camera_link bridge in sensors.launch.py),
-       so this joint is the only thing standing between the depth cloud and
-       the costmap. -->
+  <!-- RealSense D435i mounted at top of chassis at front centre -->
   <link name="camera_link">
-    <visual>
+    <!-- Camera head -->
+    <visual>
+      <origin xyz="0 0 0" rpy="0 0 0"/>
       <geometry><box size="0.025 0.09 0.025"/></geometry>
       <material name="athena_accent"/>
+    </visual>
+    <!-- Camera mount pedestal to chassis top deck -->
+    <visual>
+      <origin xyz="0 0 -0.015" rpy="0 0 0"/>
+      <geometry><box size="0.04 0.06 0.015"/></geometry>
+      <material name="athena_body"/>
     </visual>
   </link>
@@ -337,5 +337,5 @@
   <link name="gps_link">
     <visual>
-      <geometry><cylinder radius="0.035" length="0.015"/></geometry>
+      <geometry><cylinder radius="0.04" length="0.02"/></geometry>
       <material name="athena_gps"/>
     </visual>
